Commit message: fixed some of the energy-based implementation

File: urdf/irb6640_185_280.urdf (robot description, URDF)
Before this commit: robot abb_irb6640_185_280, 7 links, 6 joints
Links:
- link link_6: geometry collision mesh filename=package://abb_irb6640_support/meshes/irb6640_185_280/collis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; visual sphere radius=0.5
